Commit message: fix: Phase 2A — adapter v2, rear steering locked, friction, collision fixes
- Rewrote gazebo_cmd_vel_adapter: process cmd_vel directly in callback (no timers),
  speeds 0.05-0.60 m/s, steering 0-45deg Ackermann
- Changed rear steering joints to fixed type (no more self-steering)
- Added wheel friction mu1/mu2=1.5 for proper Ackermann grip
- Fork arms moved outward to y=±0.065/0.03, shock to side y=±0.085
- Reduced steering_link collision radius to 0.03m (avoid wheel overlap)
- Stronger steering joint damping (5.0) to prevent self-steer on spawn
- Added side parameter to corner macro for left/right mirroring

Co-Authored-By: Claude <noreply@anthropic.com>

File: src/inspection_bot_description/urdf/robot.xacro (robot description, xacro)
@@ -17,5 +17,5 @@
     wheel_center_z = steering_z + wheel_drop = -0.055 + (-0.124) = -0.179
   -->
-  <xacro:macro name="corner" params="prefix x y steering_z wheel_drop">
+  <xacro:macro name="corner" params="prefix x y steering_z wheel_drop side steering_type:=continuous">
     <!-- Steering link: servo turntable + column + fork arms + shock -->
     <link name="${prefix}_steering_link">
@@ -41,23 +41,23 @@
         <material name="dark"/>
       </visual>
-      <!-- left fork arm -->
-      <visual>
-        <origin xyz="0 0.04 -0.105" rpy="0 0 0"/>
-        <geometry>
-          <box size="0.025 0.015 0.13"/>
+      <!-- outer fork arm (farther from wheel) -->
+      <visual>
+        <origin xyz="0 ${side * 0.065} -0.105" rpy="0 0 0"/>
+        <geometry>
+          <box size="0.025 0.012 0.13"/>
         </geometry>
         <material name="grey"/>
       </visual>
-      <!-- right fork arm -->
-      <visual>
-        <origin xyz="0 -0.04 -0.105" rpy="0 0 0"/>
-        <geometry>
-          <box size="0.025 0.015 0.13"/>
+      <!-- inner fork arm (closer to wheel, but not touching) -->
+      <visual>
+        <origin xyz="0 ${side * 0.03} -0.105" rpy="0 0 0"/>
+        <geometry>
+          <box size="0.025 0.012 0.13"/>
         </geometry>
         <material name="grey"/>
       </visual>
-      <!-- simplified shock absorber / spring -->
-      <visual>
-        <origin xyz="-0.045 0 -0.095" rpy="0 0 0"/>
+      <!-- simplified shock absorber (offset to side, visual only) -->
+      <visual>
+        <origin xyz="-0.055 ${side * 0.085} -0.095" rpy="0 0 0"/>
         <geometry>
           <cylinder radius="0.012" length="0.09"/>
@@ -65,18 +65,19 @@
         <material name="orange"/>
       </visual>
+      <!-- tight collision around steering column only, avoid wheel overlap -->
       <collision>
         <origin xyz="0 0 -0.055" rpy="0 0 0"/>
         <geometry>
-          <cylinder radius="0.04" length="0.13"/>
+          <cylinder radius="0.03" length="0.08"/>
         </geometry>
       </collision>
     </link>
-    <!-- Steering joint: rotates the entire steering module around Z -->
-    <joint name="${prefix}_steering_joint" type="continuous">
+    <!-- Steering joint: strong damping prevents self-steer on spawn -->
+    <joint name="${prefix}_steering_joint" type="${steering_type}">
       <parent link="base_link"/>
       <child link="${prefix}_steering_link"/>
       <origin xyz="${x} ${y} ${steering_z}" rpy="0 0 0"/>
       <axis xyz="0 0 1"/>
-      <dynamics damping="0.5" friction="0.15"/>
+      <dynamics damping="5.0" friction="1.0"/>
     </joint>
     <!-- Wheel link -->
@@ -265,8 +266,8 @@
   </link>
   <!-- FOUR CORNERS -->
-  <xacro:corner prefix="fl" x="0.2316"  y="0.238"  steering_z="-0.055" wheel_drop="-0.124"/>
-  <xacro:corner prefix="fr" x="0.2316"  y="-0.238" steering_z="-0.055" wheel_drop="-0.124"/>
-  <xacro:corner prefix="rl" x="-0.2284" y="0.238"  steering_z="-0.055" wheel_drop="-0.124"/>
-  <xacro:corner prefix="rr" x="-0.2284" y="-0.238" steering_z="-0.055" wheel_drop="-0.124"/>
+  <xacro:corner prefix="fl" x="0.2316"  y="0.238"  steering_z="-0.055" wheel_drop="-0.124" side="1"/>
+  <xacro:corner prefix="fr" x="0.2316"  y="-0.238" steering_z="-0.055" wheel_drop="-0.124" side="-1"/>
+  <xacro:corner prefix="rl" x="-0.2284" y="0.238"  steering_z="-0.055" wheel_drop="-0.124" side="1"  steering_type="fixed"/>
+  <xacro:corner prefix="rr" x="-0.2284" y="-0.238" steering_z="-0.055" wheel_drop="-0.124" side="-1" steering_type="fixed"/>
   <!-- LIDAR -->
   <link name="lidar_link">
@@ -336,13 +337,5 @@
       <state_interface name="velocity"/>
     </joint>
-    <!-- Phase 2A: rear steering — state only, no command interface -->
-    <joint name="rl_steering_joint">
-      <state_interface name="position"/>
-      <state_interface name="velocity"/>
-    </joint>
-    <joint name="rr_steering_joint">
-      <state_interface name="position"/>
-      <state_interface name="velocity"/>
-    </joint>
+    <!-- Phase 2A: rear steering joints are fixed (not in ros2_control) -->
     <joint name="fl_wheel_joint">
       <command_interface name="velocity"/>
@@ -380,8 +373,21 @@
   <gazebo reference="rl_steering_link"><material>Gazebo/Grey</material></gazebo>
   <gazebo reference="rr_steering_link"><material>Gazebo/Grey</material></gazebo>
-  <gazebo reference="fl_wheel_link"><material>Gazebo/FlatBlack</material></gazebo>
-  <gazebo reference="fr_wheel_link"><material>Gazebo/FlatBlack</material></gazebo>
-  <gazebo reference="rl_wheel_link"><material>Gazebo/FlatBlack</material></gazebo>
-  <gazebo reference="rr_wheel_link"><material>Gazebo/FlatBlack</material></gazebo>
+  <!-- High friction for proper Ackermann steering grip -->
+  <gazebo reference="fl_wheel_link">
+    <mu1>1.5</mu1><mu2>1.5</mu2>
+    <material>Gazebo/FlatBlack</material>
+  </gazebo>
+  <gazebo reference="fr_wheel_link">
+    <mu1>1.5</mu1><mu2>1.5</mu2>
+    <material>Gazebo/FlatBlack</material>
+  </gazebo>
+  <gazebo reference="rl_wheel_link">
+    <mu1>1.5</mu1><mu2>1.5</mu2>
+    <material>Gazebo/FlatBlack</material>
+  </gazebo>
+  <gazebo reference="rr_wheel_link">
+    <mu1>1.5</mu1><mu2>1.5</mu2>
+    <material>Gazebo/FlatBlack</material>
+  </gazebo>
   <gazebo reference="lidar_link"><material>Gazebo/Blue</material></gazebo>
   <gazebo reference="camera_link"><material>Gazebo/Red</material></gazebo>

Commit message: feat: Phase 2B-1 — new inspection_bot_sim package, factory world, 2D lidar attempt
- NEW inspection_bot_sim/package (ament_python): sim launch, world, RViz
- phase2b_sim.launch.py: Gazebo + controllers + adapter + ros_gz_bridge
- phase2b_simple.sdf: factory world (ground, walls, shelves, boxes, pillar)
- phase2b_scan.rviz: RobotModel + TF + LaserScan + Odometry
- robot.xacro: added gpu_lidar sensor on lidar_link (URDF, bridge ready)
- /scan bridge connects but URDF sensor not converting in Ignition Fortress
  (future fix: standalone SDF lidar model or Ignition sensor plugin)

Co-Authored-By: Claude <noreply@anthropic.com>

File: src/inspection_bot_description/urdf/robot.xacro (robot description, xacro)
@@ -390,5 +390,28 @@
     <material>Gazebo/FlatBlack</material>
   </gazebo>
-  <gazebo reference="lidar_link"><material>Gazebo/Blue</material></gazebo>
+  <!-- Phase 2B-1: 2D Lidar sensor on lidar_link -->
+  <gazebo reference="lidar_link">
+    <material>Gazebo/Blue</material>
+    <sensor name="lidar_2d" type="gpu_lidar">
+      <always_on>true</always_on>
+      <visualize>true</visualize>
+      <update_rate>10</update_rate>
+      <lidar>
+        <scan>
+          <horizontal>
+            <samples>360</samples>
+            <resolution>1</resolution>
+            <min_angle>-3.14159</min_angle>
+            <max_angle>3.14159</max_angle>
+          </horizontal>
+        </scan>
+        <range>
+          <min>0.1</min>
+          <max>15.0</max>
+          <resolution>0.01</resolution>
+        </range>
+      </lidar>
+    </sensor>
+  </gazebo>
   <gazebo reference="camera_link"><material>Gazebo/Red</material></gazebo>
 </robot>
